Commit message: bug fixing and complete missing files for creating single_arm Tiago robot

File: Tiago/tiago_description/pmb2_description/urdf/base/base_sensors.urdf.xacro (robot description, xacro)
@@ -19,5 +19,5 @@
   <xacro:property name="base_laser_y" value="0.0"/>
   <xacro:property name="base_laser_z" value="-0.004"/>
-  <xacro:macro name="base_sensors" params=" name hokuyo:=false sick551:=false sick561:=false sick571:=false sonars:=false microphone:=false ">
+  <xacro:macro name="base_sensors" params=" name hokuyo:=false sick551:=false sick561:=false sick571:=false laser_model:=false sonars:=false microphone:=false ">
     <xacro:if value="${hokuyo}"> <!-- TODO: find expr that encure only one laser is true -->
       <!-- Laser -->

File: Tiago/tiago_description/tiago_description/robots/tiago.urdf.xacro (robot description, xacro)
@@ -13,5 +13,5 @@
     <xacro:arg name="end_effector" default="pal-hey5"/> <!-- false, pal-gripper, pal-hey5, schunk-wsg-->
     <xacro:arg name="ft_sensor" default="schunk-ft"/> <!-- false, schunk-ft -->
-    <xacro:arg name="laser_model" default="sick-571"/> <!-- false, hokuyo, sick-551, sick-561, sick-571-->
+    <xacro:arg name="laser_model" default="false"/> <!-- false, hokuyo, sick-551, sick-561, sick-571-->
     <xacro:arg name="camera_model" default="orbbec-astra"/> <!-- false, orbbec-astra, orbbec-astra-pro, asus-xtion -->
     <xacro:arg name="has_thermal_camera" default="false"/>

Commit message: Tiago Code

File: Tiago/tiago_description/pmb2_description/urdf/base/base_sensors.urdf.xacro (robot description, xacro)
@@ -19,5 +19,5 @@
   <xacro:property name="base_laser_y" value="0.0"/>
   <xacro:property name="base_laser_z" value="-0.004"/>
-  <xacro:macro name="base_sensors" params=" name hokuyo:=false sick551:=false sick561:=false sick571:=false laser_model:=false sonars:=false microphone:=false ">
+  <xacro:macro name="base_sensors" params=" name hokuyo:=false sick551:=false sick561:=false sick571:=false sonars:=false microphone:=false ">
     <xacro:if value="${hokuyo}"> <!-- TODO: find expr that encure only one laser is true -->
       <!-- Laser -->

File: Tiago/tiago_description/tiago_description/robots/tiago.urdf.xacro (robot description, xacro)
@@ -11,7 +11,7 @@
     <xacro:arg name="arm" default="true"/> <!-- true, false -->
     <xacro:arg name="wrist_model" default="wrist-2010"/>
-    <xacro:arg name="end_effector" default="pal-hey5"/> <!-- false, pal-gripper, pal-hey5, schunk-wsg-->
+    <xacro:arg name="end_effector" default="pal-gripper"/> <!-- false, pal-gripper, pal-hey5, schunk-wsg-->
     <xacro:arg name="ft_sensor" default="schunk-ft"/> <!-- false, schunk-ft -->
-    <xacro:arg name="laser_model" default="false"/> <!-- false, hokuyo, sick-551, sick-561, sick-571-->
+    <xacro:arg name="laser_model" default="sick-571"/> <!-- false, hokuyo, sick-551, sick-561, sick-571-->
     <xacro:arg name="camera_model" default="orbbec-astra"/> <!-- false, orbbec-astra, orbbec-astra-pro, asus-xtion -->
     <xacro:arg name="has_thermal_camera" default="false"/>

File: Tiago/tiago_description/tiago_description/urdf/arm/arm.urdf.xacro (robot description, xacro)
@@ -26,5 +26,5 @@
   <!-- reflect: Set to 1 for a right arm, or to -1 for a left arm-->
   <!-- tiago_dual: Set to 1 for tiago dual, -1 for original tiago, changes joints 1 and 2 -->
-  <xacro:macro name="tiago_arm" params="name parent wrist_model has_ft_sensor reflect tiago_dual *origin arm_1_offset arm_2_offset arm_3_offset arm_4_offset arm_5_offset arm_6_offset arm_7_offset">
+  <xacro:macro name="tiago_arm" params="name parent wrist_model has_ft_sensor reflect==1 tiago_dual==-1 *origin arm_1_offset arm_2_offset arm_3_offset arm_4_offset arm_5_offset arm_6_offset arm_7_offset">
     <!--************************-->
     <!--        SHOULDER        -->
