Commit message: add ur10 robot

File: UR10/cembre_description/cembre_simplified0.urdf (robot description, URDF)
Before this commit: robot sharework_simplified, 18 links, 17 joints
Links:
- added link ee_link; collision box size=0.01 0.01 0.01
- added link forearm_link, mass 3.87; collision mesh filename=/mesh/ur_e_description/meshes/ur10e/collision/forearm.stl; visual mesh filename=/mesh/ur_e_description/meshes/ur10e/visual/forearm.dae
- added link shoulder_link, mass 7.778; collision mesh filename=/mesh/ur_e_description/meshes/ur10e/collision/shoulder.stl; visual mesh filename=/mesh/ur_e_description/meshes/ur10e/visual/shoulder.dae
- added link tool0
- added link upper_arm_link, mass 12.93; collision mesh filename=/mesh/ur_e_description/meshes/ur10e/collision/upperarm.stl; visual mesh filename=/mesh/ur_e_description/meshes/ur10e/visual/upperarm.dae
- added link wrist_1_link, mass 1.96; collision mesh filename=/mesh/ur_e_description/meshes/ur10e/collision/wrist1.stl; visual mesh filename=/mesh/ur_e_description/meshes/ur10e/visual/wrist1.dae
- added link wrist_2_link, mass 1.96; collision mesh filename=/mesh/ur_e_description/meshes/ur10e/collision/wrist2.stl; visual mesh filename=/mesh/ur_e_description/meshes/ur10e/visual/wrist2.dae
- added link wrist_3_link, mass 0.202; collision mesh filename=/mesh/ur_e_description/meshes/ur10e/collision/wrist3.stl; visual mesh filename=/mesh/ur_e_description/meshes/ur10e/visual/wrist3.dae
- link base_link: mass None -> 4.0; geometry collision mesh filename=/mesh/ur_e_description/meshes/ur10e/collision/base.stl; visual mesh filename=/mesh/ur_e_description/meshes/ur10e/visual/base.dae
Joints:
- added joint ee_fixed_joint: type fixed, parent wrist_3_link, child ee_link, origin xyz=0.0 0.117 0.0 rpy=0.0 0.0 1.57079632679
- added joint elbow_joint: type revolute, parent upper_arm_link, child forearm_link, origin xyz=0.0 -0.137 0.613 rpy=0.0 0.0 0.0, axis 0 1 0, limit lower=-3.14159265359 upper=3.14159265359 effort=150.0 velocity=3.14
- added joint shoulder_lift_joint: type revolute, parent shoulder_link, child upper_arm_link, origin xyz=0.0 0.176 0.0 rpy=0.0 1.57079632679 0.0, axis 0 1 0, limit lower=-3.14159265359 upper=0.052359878 effort=330.0 velocity=3.14
- added joint shoulder_pan_joint: type revolute, parent base_link, child shoulder_link, origin xyz=0.0 0.0 0.181 rpy=0.0 0.0 0.0, axis 0 0 1, limit lower=-3.14159265359 upper=3.14159265359 effort=330.0 velocity=3.14
- added joint wrist_1_joint: type revolute, parent forearm_link, child wrist_1_link, origin xyz=0.0 0.0 0.571 rpy=0.0 1.57079632679 0.0, axis 0 1 0, limit lower=-3.14159265359 upper=3.14159265359 effort=54.0 velocity=6.28
- added joint wrist_2_joint: type revolute, parent wrist_1_link, child wrist_2_link, origin xyz=0.0 0.135 0.0 rpy=0.0 0.0 0.0, axis 0 0 1, limit lower=-3.14159265359 upper=3.14159265359 effort=54.0 velocity=6.28
- added joint wrist_3_joint: type revolute, parent wrist_2_link, child wrist_3_link, origin xyz=0.0 0.0 0.12 rpy=0.0 0.0 0.0, axis 0 1 0, limit lower=-6.28318530718 upper=6.28318530718 effort=54.0 velocity=6.28
- added joint wrist_3_link-tool0_fixed_joint: type fixed, parent wrist_3_link, child tool0, origin xyz=0 0.117 0 rpy=-1.57079632679 0 0
